Commit message: lidar with no cable, color parameters launch

File: urdf/lite3/lite.urdf.xacro (robot description, xacro)
@@ -6,4 +6,5 @@
         box_color
         pi_module_color
+        spacers_color
         raspy_color
         lidar_color
@@ -36,7 +37,7 @@
         <link name="${prefix}pi_module_link">
             <visual>
-                <origin xyz="0 0 0" rpy="${pi/2} 0 ${pi/2}"/>
+                <origin xyz="0 0 0" rpy="0 0 ${-pi/2}"/>
                 <geometry>
-                    <mesh filename="file://$(find robotont_lite_description)/meshes/lite3/pi_module.STL"/>
+                    <mesh filename="file://$(find robotont_lite_description)/meshes/lite3/pi_module_pla.STL"/>
                 </geometry>
                 <material name="${prefix}pi_module_material">
@@ -50,5 +51,25 @@
             <axis xyz="0 0 0"/>
             <origin
-                xyz="-0.073 -0.065 ${cable_box_elevation}"
+                xyz="0.015 0 ${cable_box_elevation}"
+                rpy="0 0 0"
+            />
+        </joint>
+        <link name="${prefix}pi_module_spacers_link">
+            <visual>
+                <origin xyz="0 0 0" rpy="0 0 ${-pi/2}"/>
+                <geometry>
+                    <mesh filename="file://$(find robotont_lite_description)/meshes/lite3/pi_module_spacers.STL"/>
+                </geometry>
+                <material name="${prefix}pi_module_spacers_material">
+                    <color rgba="${spacers_color}"/>
+                </material>
+            </visual>
+        </link>
+        <joint name="${prefix}pi_module_spacers_joint" type="fixed">
+            <parent link="${prefix}base_link"/>
+            <child link="${prefix}pi_module_spacers_link"/>
+            <axis xyz="0 0 0"/>
+            <origin
+                xyz="0.015 0 ${cable_box_elevation}"
                 rpy="0 0 0"
             />
@@ -79,5 +100,5 @@
                 <origin xyz="0 0 0" rpy="${pi/2} 0 ${pi}"/>
                 <geometry>
-                    <mesh filename="file://$(find robotont_lite_description)/meshes/lite3/rplidar-a2m4-r1.STL"/>
+                    <mesh scale="0.001 0.001 0.001" filename="file://$(find robotont_lite_description)/meshes/lite3/rplidar-a2m4-r1_no_cable.STL"/>
                 </geometry>
                 <material name="${prefix}lidar_material">
@@ -91,6 +112,26 @@
             <axis xyz="0 0 0"/>
             <origin
-                xyz="0.065 -0.047 ${cable_box_elevation+0.053}"
+                xyz="0.065 -0.047 ${cable_box_elevation+0.049}"
                 rpy="0 0 0"
+            />
+        </joint>
+        <link name="${prefix}camera_link">
+            <visual>
+                <origin xyz="0 0 0" rpy="${pi/2} 0 ${pi/2}"/>
+                <geometry>
+                    <mesh scale="0.001 0.001 0.001" filename="file://$(find robotont_lite_description)/meshes/lite3/rpiAIcamera.STL"/>
+                </geometry>
+                <material name="${prefix}camera_material">
+                    <color rgba="${lidar_color}"/>
+                </material>
+            </visual>
+        </link>
+        <joint name="${prefix}camera_joint" type="fixed">
+            <parent link="${prefix}base_link"/>
+            <child link="${prefix}camera_link"/>
+            <axis xyz="0 0 0"/>
+            <origin
+                xyz="0.06 -0.011 ${cable_box_elevation+0.005}"
+                rpy="0 -0.08 0"
             />
         </joint>

File: urdf/lite3/robotont_lite.urdf.xacro (robot description, xacro)
@@ -1,10 +1,10 @@
 <?xml version="1.0"?>
 <robot xmlns:xacro="http://ros.org/wiki/xacro" name="robotont_lite">
+    <xacro:property name="primary_color" value="$(arg main_color)"/>
+    <xacro:property name="secondary_color" value="$(arg second_color)"/>
     <xacro:include filename="$(find robotont_description)/urdf/gen3/robotont.urdf.xacro"/>
     <xacro:include filename="$(find robotont_description)/urdf/gen3/base.urdf.xacro"/>
     <xacro:include filename="$(find robotont_description)/urdf/gen3/motor.urdf.xacro"/>
     <xacro:include filename="$(find robotont_lite_description)/urdf/lite3/lite.urdf.xacro"/>
-    <xacro:property name="cable_box_color" value="1.0 1.0 0.0 1.0"/>
-    <xacro:property name="pi_module_color" value="1.0 1.0 0.0 1.0"/>
     <xacro:property name="raspy_color" value="0 0.55 0.29 1.0"/>
     <xacro:property name="lidar_color" value="0.26 0.26 0.26 1.0"/>
@@ -12,6 +12,7 @@
     <xacro:lite_macro
         prefix="${prefix}"
-        box_color="${cable_box_color}"
-        pi_module_color="${pi_module_color}"
+        box_color="${secondary_color}"
+        pi_module_color="${secondary_color}"
+        spacers_color="${spacers_color}"
         raspy_color="${raspy_color}"
         lidar_color="${lidar_color}"

Commit message: loading meshes using the package substitute to make it work also for distributed ros

File: urdf/lite3/lite.urdf.xacro (robot description, xacro)
@@ -19,5 +19,5 @@
                 <origin xyz="0 -0.043 0" rpy="${pi/2} 0 ${pi/2}"/>
                 <geometry>
-                    <mesh filename="file://$(find robotont_lite_description)/meshes/lite3/cable_box.STL"/>
+                    <mesh filename="package://robotont_lite_description/meshes/lite3/cable_box.STL"/>
                 </geometry>
                 <material name="${prefix}cable_box_material">
@@ -39,5 +39,5 @@
                 <origin xyz="0 0 0" rpy="0 0 ${-pi/2}"/>
                 <geometry>
-                    <mesh filename="file://$(find robotont_lite_description)/meshes/lite3/pi_module_pla.STL"/>
+                    <mesh filename="package://robotont_lite_description/meshes/lite3/pi_module_pla.STL"/>
                 </geometry>
                 <material name="${prefix}pi_module_material">
@@ -59,5 +59,5 @@
                 <origin xyz="0 0 0" rpy="0 0 ${-pi/2}"/>
                 <geometry>
-                    <mesh filename="file://$(find robotont_lite_description)/meshes/lite3/pi_module_spacers.STL"/>
+                    <mesh filename="package://robotont_lite_description/meshes/lite3/pi_module_spacers.STL"/>
                 </geometry>
                 <material name="${prefix}pi_module_spacers_material">
@@ -79,5 +79,5 @@
                 <origin xyz="0 0 0" rpy="0 0 ${pi}"/>
                 <geometry>
-                    <mesh filename="file://$(find robotont_lite_description)/meshes/lite3/RPi_case.STL"
+                    <mesh filename="package://robotont_lite_description/meshes/lite3/RPi_case.STL"
                     scale="0.001 0.001 0.001"/>
                 </geometry>
@@ -100,5 +100,5 @@
                 <origin xyz="0 0 0" rpy="${pi/2} 0 ${pi}"/>
                 <geometry>
-                    <mesh scale="0.001 0.001 0.001" filename="file://$(find robotont_lite_description)/meshes/lite3/rplidar-a2m4-r1_no_cable.STL"/>
+                    <mesh scale="0.001 0.001 0.001" filename="package://robotont_lite_description/meshes/lite3/rplidar-a2m4-r1_no_cable.STL"/>
                 </geometry>
                 <material name="${prefix}lidar_material">
@@ -120,5 +120,5 @@
                 <origin xyz="0 0 0" rpy="${pi/2} 0 ${pi/2}"/>
                 <geometry>
-                    <mesh scale="0.001 0.001 0.001" filename="file://$(find robotont_lite_description)/meshes/lite3/rpiAIcamera.STL"/>
+                    <mesh scale="0.001 0.001 0.001" filename="package://robotont_lite_description/meshes/lite3/rpiAIcamera.STL"/>
                 </geometry>
                 <material name="${prefix}camera_material">

Commit message: added laser_link for lidar with corrected orientation

File: urdf/lite3/lite.urdf.xacro (robot description, xacro)
@@ -98,5 +98,5 @@
         <link name="${prefix}lidar_link">
             <visual>
-                <origin xyz="0 0 0" rpy="${pi/2} 0 ${pi}"/>
+                <origin xyz="0.065 -0.047 0" rpy="${pi/2} 0 ${pi}"/>
                 <geometry>
                     <mesh scale="0.001 0.001 0.001" filename="package://robotont_lite_description/meshes/lite3/rplidar-a2m4-r1_no_cable.STL"/>
@@ -110,9 +110,11 @@
             <parent link="${prefix}base_link"/>
             <child link="${prefix}lidar_link"/>
-            <axis xyz="0 0 0"/>
-            <origin
-                xyz="0.065 -0.047 ${cable_box_elevation+0.049}"
-                rpy="0 0 0"
-            />
+            <origin xyz="0 0 ${cable_box_elevation+0.049}" rpy="0 0 0"/>
+        </joint>
+        <link name="${prefix}laser_link"/>
+        <joint name="${prefix}laser_joint" type="fixed">
+            <parent link="${prefix}lidar_link"/>
+            <child link="${prefix}laser_link"/>
+            <origin xyz="0 0 0.035" rpy="0 0 ${pi}"/>
         </joint>
         <link name="${prefix}camera_link">
